Commit message: Se estructura correctamente el URDF con información para su interpretación en salon de clase

File: urdf/scorbot.urdf (robot description, URDF)
Before this commit: robot scorbot, 7 links, 6 joints
Joints:
- joint j4: origin xyz=0.22 0.0 0.0 rpy=0 0 1.57 -> xyz=0.22 0.0 0.00 rpy=0 0 1.57
